File: pc_cooler/PC temperature Monitor.brd (EAGLE design)
At the start: 68.6 x 53.3 mm, 6 parts

Commit message: Add files via upload
Parts:
- added MDC Motor- 12v: (no value), AUTODESK_CIRCUITS_BREADBOARD:2P-2.54-65/35MIL
- added Ppower supply: 12V, AUTODESK_CIRCUITS_BREADBOARD:2P-2.54-65/35MIL
- added QTIP120: (no value), AUTODESK_CIRCUITS_BREADBOARD:TO220
- added Resister: 2.2k‎Ω, AUTODESK_CIRCUITS_BREADBOARD:0207/10
- renumbered R-Resistor to Resistor, Rpot-potentiometer to Rpotentiometer
Connections:
- removed net N$10 (its old number): Rpot-Touch sensor.E, Rpotentiometer.A, U-Arduino Uno R3.GND.., U-DTH11/TMP36.1, U-LCD 16X2 display.1, U-LCD 16X2 display.16, U-LCD 16X2 display.5
- new net N$16: Resister.1, U-Arduino Uno R3.8
- new net N$17: MDC Motor- 12v.2, Ppower supply.2
- new net N$18: MDC Motor- 12v.1, QTIP120.2
- new net N$19: Ppower supply.1, QTIP120.3, Rpot-Touch sensor.E, Rpotentiometer.A, U-Arduino Uno R3.GND.., U-DTH11/TMP36.1, U-LCD 16X2 display.1, U-LCD 16X2 display.16, U-LCD 16X2 display.5
- new net N$20: QTIP120.1, Resister.2
